Commit message: add ORB SLAM configuration

File: robot_learning/urdf/robot.xacro (robot description, xacro)
@@ -110,5 +110,5 @@
         <parent link="chassis"/>
         <child link="camera"/>
-        <origin xyz="${0.1-3*inch} 0 0.1" rpy="0 0 0"/>
+        <origin xyz="0.05 0 0.1" rpy="0 0 0"/>
     </joint>
 	<link name="camera_optical"/>

Commit message: fix robot model + more configurations

File: robot_learning/urdf/robot.xacro (robot description, xacro)
@@ -64,5 +64,5 @@
         <origin xyz="0 ${-wd/2} ${wr}" rpy="${-pi/2} 0 0"/>
     </xacro:wheel>
-    <link name="caster">
+    <link name="front_caster">
         <inertial>
             <mass value="0.1"/>
@@ -84,8 +84,33 @@
         </collision>
     </link>
-    <joint name="caster_joint" type="fixed">
+    <joint name="front_caster_joint" type="fixed">
         <origin xyz="${5.0*inch} 0 ${3.0/2*inch}" rpy="0 0 0"/>
         <parent link="base_link"/>
-        <child link="caster"/>
+        <child link="front_caster"/>
+    </joint>
+    <link name="back_caster">
+        <inertial>
+            <mass value="0.1"/>
+            <sphere radius="${3.0/2 * inch}"/>
+            <sphere_inertia m="0.1" r="${3.0/2 * inch}"/>
+        </inertial>
+        <visual>
+            <geometry>
+                <sphere radius="${3.0/2 * inch}"/>
+            </geometry>
+            <material name="black">
+                <color rgba="0 0 0 0.5"/>
+            </material>
+        </visual>
+        <collision>
+            <geometry>
+                <sphere radius="${3.0/2 * inch}"/>
+            </geometry>
+        </collision>
+    </link>
+    <joint name="back_caster_joint" type="fixed">
+        <origin xyz="${-3.0*inch} 0 ${3.0/2*inch}" rpy="0 0 0"/>
+        <parent link="base_link"/>
+        <child link="back_caster"/>
     </joint>
     <link name="camera">
@@ -121,14 +146,14 @@
         <inertial>
             <mass value="0.1"/>
-            <cylinder_inertia m="0.1" r="${4*inch}" h="${0.1*inch}"/>
+            <cylinder_inertia m="0.1" r="${2*inch}" h="${0.1*inch}"/>
         </inertial>
         <visual>
             <geometry>
-                <cylinder length="${0.1*inch}" radius="${4*inch}"/>
+                <cylinder length="${0.1*inch}" radius="${2*inch}"/>
             </geometry>
         </visual>
         <collision>
             <geometry>
-                <cylinder length="${0.1*inch}" radius="${4*inch}"/>
+                <cylinder length="${0.1*inch}" radius="${2*inch}"/>
             </geometry>
         </collision>
@@ -137,5 +162,5 @@
         <parent link="base_link"/>
         <child link="base_laser_link"/>
-        <origin xyz="${-3*inch} 0 ${2.5 * inch + 0.1 * inch}" rpy="0 0 -3.14"/>
+        <origin xyz="${-3*inch} 0 ${2.5 * inch + 0.8 * inch}" rpy="0 0 -3.14"/>
     </joint>
 </robot>

Commit message: absolute confusion with new pipeline - may re-impl

File: robot_learning/urdf/robot.xacro (robot description, xacro)
@@ -135,5 +135,5 @@
         <parent link="chassis"/>
         <child link="camera"/>
-        <origin xyz="0.05 0 0.1" rpy="0 0 0"/>
+        <origin xyz="0.15 0 0.1" rpy="0 0 0"/>
     </joint>
 	<link name="camera_optical"/>

Commit message: update report

File: robot_learning/urdf/robot.xacro (robot description, xacro)
@@ -135,9 +135,9 @@
         <parent link="chassis"/>
         <child link="camera"/>
-        <origin xyz="0.15 0 0.1" rpy="0 0 0"/>
+        <origin xyz="0.25 0 0.1" rpy="0 0 0"/>
     </joint>
 	<link name="camera_optical"/>
 	<joint name="camera_optical_joint" type="fixed">
-		<origin xyz="0 0 0" rpy="${-pi/2} 0 ${-pi/2}"/>
+		<origin xyz="0 0 0" rpy="${-pi/2 - 30*deg} 0 ${-pi/2}"/>
         <parent link="camera"/>
         <child link="camera_optical"/>

Commit message: turns out camera pitch was not configured correctly

File: robot_learning/urdf/robot.xacro (robot description, xacro)
@@ -135,9 +135,9 @@
         <parent link="chassis"/>
         <child link="camera"/>
-        <origin xyz="0.25 0 0.1" rpy="0 0 0"/>
+        <origin xyz="0.25 0 0.1" rpy="0 ${-30*deg} 0"/>
     </joint>
 	<link name="camera_optical"/>
 	<joint name="camera_optical_joint" type="fixed">
-		<origin xyz="0 0 0" rpy="${-pi/2 - 30*deg} 0 ${-pi/2}"/>
+		<origin xyz="0 0 0" rpy="${-pi/2} 0 ${-pi/2}"/>
         <parent link="camera"/>
         <child link="camera_optical"/>

Commit message: stable for now

File: robot_learning/urdf/robot.xacro (robot description, xacro)
@@ -135,5 +135,5 @@
         <parent link="chassis"/>
         <child link="camera"/>
-        <origin xyz="0.25 0 0.1" rpy="0 ${-30*deg} 0"/>
+        <origin xyz="0.25 0 0.1" rpy="0 ${10*deg} 0"/>
     </joint>
 	<link name="camera_optical"/>

Commit message: sideways-camera configuration (WARNING :: required to FIX ALL of T_b2c / URDF / ymin parametrization)

File: robot_learning/urdf/robot.xacro (robot description, xacro)
@@ -135,5 +135,5 @@
         <parent link="chassis"/>
         <child link="camera"/>
-        <origin xyz="0.25 0 0.1" rpy="0 ${10*deg} 0"/>
+        <origin xyz="0.25 0.25 0.1" rpy="0 ${10*deg} ${90*deg}"/>
     </joint>
 	<link name="camera_optical"/>

Commit message: fixed perplexing scale issue + lots of heuristics around the architecture

File: robot_learning/urdf/robot.xacro (robot description, xacro)
@@ -135,5 +135,5 @@
         <parent link="chassis"/>
         <child link="camera"/>
-        <origin xyz="0.25 0.25 0.1" rpy="0 ${10*deg} ${90*deg}"/>
+        <origin xyz="0.25 0.25 0.1" rpy="0 0 0"/>
     </joint>
 	<link name="camera_optical"/>
